File: kfet-elec-ruler/kfet-elec-ruler.kicad_pcb (KiCad board)
At the start: 2 copper layers, 160 x 40 mm, 51 parts

Commit message: WIP
Parts:
- added REF**: R_0201_0603Metric, Resistor_SMD:R_0201_0603Metric, F.Cu at (163.8, 88.3)
- moved 0402 71.8 mm to (163.8, 85.7)
- moved 0603 71.8 mm to (163.8, 83.2)
- moved 0805 71.8 mm to (163.8, 80.6)
- moved 1206 71.8 mm to (163.8, 77.5)
- moved 1812 71.8 mm to (163.8, 69.2)
- moved 2010 71.8 mm to (163.8, 73.7)
- moved 2512 71.8 mm to (163.8, 64.1)
- moved AWG Gauge 2.50 mm to (176.5, 86.0)
Routing:
- net (no net): track 115.6 -> 126.6 mm
Other:
- net class .2 removed
- net class .3 removed
- net class .4 removed
- net class .5 removed
- net class .75 removed
- net class 1 removed
- net class 1.25 removed
- net class 2.0 removed
- net class 2.5 removed
- net class Default removed
- board text added: "0.10mm"
- board text added: "0201"
- board text added: "I max (+10°C)"
- board text removed: "1 Croque : 1,5€"
- board text removed: "10 Croques : 10€"
- board text removed: "2 Croques : 2,5€"
- board text removed: "Blanche : 1,0€"
- board text removed: "Café : 0,5€"
- board text removed: "KFet Élec 2019-2020"
- board text removed: "SMD footprints"
- board text removed: "Soft : 0,9€"
- board text removed: "Val-Dieu : 1,5€"
- board text removed: "~~~~Entre le R3 et le R7~~~~"
